File: hardware/uno-analog-input/uno-analog-input.kicad_pcb (KiCad board)
At the start: 2 copper layers, 68.6 x 53.3 mm, 23 parts, among them J1 PinHeader_02x06_2.54mm, P1 Power, P2 Analog, P3 Digital, P4 Digital, P5 CONN_01X01, P6 CONN_01X01, P7 CONN_01X01, P8 CONN_01X01

Commit message: upload modified file
Parts:
- removed C1, C2, C3, C4, C5, C6: 22p, Capacitor_THT:C_Disc_D4.3mm_W1.9mm_P5.00mm
- added R10: 1M, Resistor_THT:R_Axial_DIN0204_L3.6mm_D1.6mm_P7.62mm_Horizontal, F.Cu at (154.2, 101.0)
- added R12: 1M, Resistor_THT:R_Axial_DIN0204_L3.6mm_D1.6mm_P7.62mm_Horizontal, F.Cu at (154.2, 106.0)
- added R5: 1M, Resistor_THT:R_Axial_DIN0204_L3.6mm_D1.6mm_P7.62mm_Horizontal, F.Cu at (138.9, 103.5)
- added R7: 1M, Resistor_THT:R_Axial_DIN0204_L3.6mm_D1.6mm_P7.62mm_Horizontal, F.Cu at (154.2, 93.3)
- added R8: 1M, Resistor_THT:R_Axial_DIN0204_L3.6mm_D1.6mm_P7.62mm_Horizontal, F.Cu at (154.2, 95.9)
- added R9: 1M, Resistor_THT:R_Axial_DIN0204_L3.6mm_D1.6mm_P7.62mm_Horizontal, F.Cu at (154.2, 98.4)
- moved R11 16.5 mm to (154.2, 103.5)
- moved G2 2.54 mm to (165.6, 99.7)
- moved R1 1.27 mm to (138.9, 93.3)
- moved R2 1.27 mm to (138.9, 95.9)
- moved R3 1.27 mm to (138.9, 98.4)
- moved R4 1.27 mm to (138.9, 101.0)
- moved R6 1.27 mm to (138.9, 106.0)
- renumbered R5 to R11
Connections:
- R1 pad 1: /A5(SCL) -> GND
- R2 pad 1: /A4(SDA) -> GND
- R3 pad 1: /A3 -> GND
- R4 pad 1: /A2 -> GND
- R6 pad 1: /A0 -> GND
Routing:
- net /A5(SCL): track 78.6 -> 121.5 mm
- net GND: track 106.0 -> 87.2 mm
- net Net-(J1-Pad8): track 5.08 -> 22.5 mm
- net Net-(J1-Pad6): track 5.08 -> 22.5 mm
- net Net-(J1-Pad12): track 5.08 -> 22.5 mm
- net Net-(J1-Pad10): track 5.08 -> 22.5 mm
- net Net-(J1-Pad2): track 5.08 -> 22.5 mm
- net Net-(J1-Pad4): track 5.08 -> 22.5 mm
- net /A3: track 48.2 -> 31.7 mm
- net /A2: track 43.3 -> 28.1 mm
- net /A1: track 39.6 -> 24.5 mm
- net /A0: track 35.2 -> 20.9 mm
- net /A4(SDA): track 75.1 -> 65.6 mm
- added copper zone on F.Cu, net GND
- removed copper zone on B.Cu, net GND
Other:
- board text added: "GND"
- board text added: "IN"
