File: hardware/uno-analog-input/uno-analog-input.sch (KiCad schematic (older format))
At the start: 23 parts, among them J1 PinHeader_02x06_2.54mm, P1 Power, P2 Analog, P3 Digital, P4 Digital, P5 CONN_01X01, P6 CONN_01X01, P7 CONN_01X01, P8 CONN_01X01

Commit message: upload modified file
Parts:
- removed C1, C2, C3, C4, C5, C6: 22p, Capacitor_THT:C_Disc_D4.3mm_W1.9mm_P5.00mm, symbol Device:C
- added R10, R12, R5, R7, R8, R9: 1M, Resistor_THT:R_Axial_DIN0204_L3.6mm_D1.6mm_P7.62mm_Horizontal, symbol Device:R
- renumbered R5 to R11
Other:
- moved on the sheet: R11
